Commit message: prepare for test on the real robot

File: description/camera.xacro (robot description, xacro)
@@ -1,13 +1,18 @@
 <?xml version="1.0"?>
 <robot xmlns:xacro="http://www.ros.org/wiki/xacro" >
+    <xacro:property name="camera_length" value="0.010"/>
+    <xacro:property name="camera_width" value="0.03"/>
+    <xacro:property name="camera_height" value="0.03"/>
+    <xacro:property name="camera_offset_x" value="${chassis_length - camera_length/2}"/>
+    <xacro:property name="camera_offset_z" value="${camera_height/2 + chassis_height}"/>
     <joint name="camera_joint" type="fixed">
         <parent link="chassis"/>
         <child link="camera_link"/>
-        <origin xyz="0.21 0 0.02" rpy="0 0 0"/>
+        <origin xyz="${camera_offset_x} 0 ${camera_offset_z}" rpy="0 0 0"/>
     </joint>
     <link name="camera_link">
         <visual>
             <geometry>
-                <box size="0.010 0.03 0.03"/>
+                <box size="${camera_length} ${camera_width} ${camera_height}"/>
             </geometry>
             <material name="black"/>

File: description/robot.urdf.xacro (robot description, xacro)
@@ -2,6 +2,10 @@
 <robot xmlns:xacro="http://www.ros.org/wiki/xacro"  name="robot">
     <xacro:include filename="robot_core.xacro" />
-    <!-- <xacro:include filename="gazebo_control.xacro" /> -->
-    <xacro:include filename="ros2_control.xacro" />
     <xacro:include filename="camera.xacro" />
+    <xacro:if value="$(arg use_ros2_control)">
+        <xacro:include filename="ros2_control.xacro" />
+    </xacro:if>
+    <xacro:unless value="$(arg use_ros2_control)">
+        <xacro:include filename="gazebo_control.xacro" />
+    </xacro:unless>
 </robot>

File: description/robot_core.xacro (robot description, xacro)
@@ -2,4 +2,19 @@
 <robot xmlns:xacro="http://www.ros.org/wiki/xacro"  name="robot">
     <xacro:include filename="inertial_macros.xacro" />
+    <!-- Config the dimensions -->
+    <xacro:property name="chassis_length" value="0.21"/>
+    <xacro:property name="chassis_width" value="0.1"/>
+    <xacro:property name="chassis_height" value="0.02"/>
+    <xacro:property name="chassis_mass" value="0.5"/>
+    <xacro:property name="wheel_radius" value="0.0375"/>
+    <xacro:property name="wheel_thickness" value="0.03"/>
+    <xacro:property name="wheel_mass" value="0.1"/>
+    <xacro:property name="wheel_offset_x" value="0.075"/>
+    <xacro:property name="wheel_offset_y" value="0.065"/>
+    <xacro:property name="wheel_offset_z" value="0"/>
+    <xacro:property name="caster_wheel_radius" value="0.015"/>
+    <xacro:property name="caster_wheel_mass" value="0.1"/>
+    <xacro:property name="caster_wheel_offset_x" value="0.185"/>
+    <xacro:property name="caster_wheel_offset_z" value="${caster_wheel_radius}"/>
 <!-- SETTING MATERIALS -->
     <material name="white">
@@ -22,22 +37,22 @@
         <parent link="base_link"/>
         <child link="chassis"/>
-        <origin xyz="-0.075 0 0"/>
+        <origin xyz="${-wheel_offset_x} 0 ${-wheel_offset_z}"/>
     </joint>
     <link name="chassis">
         <visual>
-            <origin xyz="0.105 0 0.0025" rpy="0 0 0"/>
+            <origin xyz="${chassis_length/2} 0 ${chassis_height/2}"/>
             <geometry>
-                <box size="0.21 0.1 0.02"/>
+                <box size="${chassis_length} ${chassis_width} ${chassis_height}"/>
             </geometry>
             <material name="white"/>
         </visual>
         <collision>
-            <origin xyz="0.105 0 0.0025" rpy="0 0 0"/>
+            <origin xyz="${chassis_length/2} 0 ${chassis_height/2}"/>
             <geometry>
-                <box size="0.21 0.1 0.02"/>
+                <box size="${chassis_length} ${chassis_width} ${chassis_height}"/>
             </geometry>
         </collision>
-        <xacro:inertial_box mass="0.5" x="0.21" y="0.1" z="0.02">
-            <origin xyz="0.105 0 0.0025" rpy="0 0 0"/>
+        <xacro:inertial_box mass="${chassis_mass    }" x="${chassis_length}" y="${chassis_width}" z="${chassis_height}">
+            <origin xyz="${chassis_length/2} 0 ${chassis_height/2}" rpy="0 0 0"/>
         </xacro:inertial_box>
     </link>
@@ -46,5 +61,5 @@
         <parent link="base_link"/>
         <child link="left_wheel"/>
-        <origin xyz="0 0.065 0" rpy="-${pi/2} 0 0"/>
+        <origin xyz="0 ${wheel_offset_y} 0" rpy="-${pi/2} 0 0" />
         <axis xyz="0 0 1"/>
     </joint>
@@ -52,5 +67,5 @@
         <visual>
             <geometry>
-                <cylinder length="0.03" radius="0.0375" />
+                <cylinder radius="${wheel_radius}" length="${wheel_thickness}"/>
             </geometry>
             <material name="black"/>
@@ -58,8 +73,8 @@
         <collision>
             <geometry>
-                <cylinder length="0.03" radius="0.0375" />
+                <sphere radius="${wheel_radius}"/>
             </geometry>
         </collision>
-        <xacro:inertial_cylinder mass="0.1" length="0.03" radius="0.0375">
+        <xacro:inertial_cylinder mass="${wheel_mass}" length="${wheel_thickness}" radius="${wheel_radius}">
             <origin xyz="0 0 0" rpy="0 0 0"/>
         </xacro:inertial_cylinder>
@@ -69,5 +84,5 @@
         <parent link="base_link"/>
         <child link="right_wheel"/>
-        <origin xyz="0 -0.065 0" rpy="${pi/2} 0 0"/>
+        <origin xyz="0 ${-wheel_offset_y} 0" rpy="${pi/2} 0 0"/>
         <axis xyz="0 0 -1"/>
     </joint>
@@ -75,5 +90,5 @@
         <visual>
             <geometry>
-                <cylinder length="0.03" radius="0.0375" />
+                <cylinder radius="${wheel_radius}" length="${wheel_thickness}"/>
             </geometry>
             <material name="black"/>
@@ -81,8 +96,8 @@
         <collision>
             <geometry>
-                <cylinder length="0.03" radius="0.0375" />
+                <sphere radius="${wheel_radius}"/>
             </geometry>
         </collision>
-        <xacro:inertial_cylinder mass="0.1" length="0.03" radius="0.0375">
+        <xacro:inertial_cylinder mass="${wheel_mass}" length="${wheel_thickness}" radius="${wheel_radius}">
             <origin xyz="0 0 0" rpy="0 0 0"/>
         </xacro:inertial_cylinder>
@@ -92,10 +107,10 @@
         <parent link="chassis"/>
         <child link="caster_wheel"/>
-        <origin xyz="0.185 0 -0.0225" rpy="0 0 0"/>
+        <origin xyz="${caster_wheel_offset_x} 0 ${-caster_wheel_offset_z}"/>
     </joint>
     <link name="caster_wheel">
         <visual>
             <geometry>
-                <sphere radius="0.015" />
+                <sphere radius="${caster_wheel_radius}"/>
             </geometry>
             <material name="blue"/>
@@ -103,8 +118,8 @@
         <collision>
             <geometry>
-                <sphere radius="0.015" />
+                <sphere radius="${caster_wheel_radius}"/>
             </geometry>
         </collision>
-        <xacro:inertial_sphere mass="0.1" radius="0.015">
+        <xacro:inertial_sphere mass="${caster_wheel_mass}" radius="${caster_wheel_radius}">
             <origin xyz="0 0 0" rpy="0 0 0"/>
         </xacro:inertial_sphere>
